File: kicad/SuperPSU_C64.kicad_pcb (KiCad board)
At the start: 4 copper layers, 80 x 75.5 mm, 35 parts, among them J1 9VAC, J2 9VAC, J3 5VDC, J4 9VAC, J5 14VDC, Q1 TIC116, U1 TSR3-2450N

Commit message: Add files via upload
Parts:
- D6: value P6Ke15CA -> D_TVS
- moved D6 10.2 mm to (79.2, 98.1), turned to 90 degrees
Connections:
- D6 pad 1: Net-(D4-A) -> Net-(D6-A1)
- D6 pad 2: Net-(D6-A) -> Net-(D4-A)
- J2 pad 1: Net-(D6-A) -> Net-(D6-A1)
- J4 pad 2: Net-(D6-A) -> Net-(D6-A1)
- R4 pad 2: Net-(D6-A) -> Net-(D6-A1)
Routing:
- net Net-(D6-A1): vias 0 -> 45
- net Net-(D6-A): vias 45 -> 0
- added copper zone on B.Cu, net Net-(D6-A1)
- added copper zone on F.Cu, net Net-(D6-A1)
- added copper zone on In1.Cu, net Net-(D6-A1)
- added copper zone on In2.Cu, net Net-(D6-A1)
- removed copper zone on B.Cu, net Net-(D6-A)
- removed copper zone on F.Cu, net Net-(D6-A)
- removed copper zone on In1.Cu, net Net-(D6-A)
- removed copper zone on In2.Cu, net Net-(D6-A)
